File: temp_room_module_wireless.brd (EAGLE design)
At the start: 7.2 x 7.1 mm, 58 parts, among them IC3 DS1307, J7 ICSP, Q1 32.768

Commit message: updates and stencil
Routing:
- net S$89: track 0.00 -> 23.6 mm
- net S$16: track 9.07 -> 0.00 mm
- net S$75: track 0.00 -> 6.47 mm
- net GND: track 357.7 -> 360.3 mm
- removed copper zone on layer 1, net GND
- removed copper zone on layer 16, net GND
Changed lines of the file:
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@@
 <?xml version="1.0" encoding="utf-8"?>
 <!DOCTYPE eagle SYSTEM "eagle.dtd">
-<eagle version="6.1">
+<eagle version="6.4">
 <drawing>
 <settings>
@@
 <setting verticaltext="up"/>
 </settings>
-<grid distance="1" unitdist="mm" unit="mm" style="lines" multiple="1" display="yes" altdistance="0.025" altunitdist="inch" altunit="inch"/>
+<grid distance="0.1" unitdist="mm" unit="mm" style="lines" multiple="1" display="yes" altdistance="0.025" altunitdist="inch" altunit="inch"/>
 <layers>
 <layer number="1" name="Top" color="4" fill="1" visible="yes" active="yes"/>
@@
 </class>
 </classes>
-<designrules>
+<designrules name="default">
 <description language="de">&lt;b&gt;EAGLE Design Rules&lt;/b&gt;
 &lt;p&gt;
@@
 <signal name="S$20">
 </signal>
+<signal name="S$75">
+<wire x1="4" y1="21.6" x2="6.7" y2="18.9" width="0.4064" layer="16"/>
+<wire x1="3.4" y1="24" x2="3.4" y2="22.2" width="0.4064" layer="16"/>
+<wire x1="3.4" y1="22.2" x2="4" y2="21.6" width="0.4064" layer="16"/>
+</signal>
 <signal name="GND">
 <wire x1="42.4" y1="72" x2="42.4" y2="61.6" width="0.4064" layer="1"/>
@@
 <wire x1="42.2" y1="29.1" x2="42.2" y2="29" width="0.4064" layer="16"/>
 <wire x1="42.2" y1="29" x2="40" y2="26.8" width="0.4064" layer="16"/>
-<wire x1="6.6" y1="19" x2="7.6" y2="19" width="0.4064" layer="16"/>
-<wire x1="7.6" y1="19" x2="9.6" y2="21" width="0.4064" layer="16"/>
-<wire x1="9.6" y1="25.2" x2="9.6" y2="24" width="0.4064" layer="16"/>
-<wire x1="9.6" y1="24" x2="9.6" y2="21" width="0.4064" layer="16"/>
-<wire x1="3.9" y1="32.1" x2="3.9" y2="30.9" width="0.4064" layer="1"/>
-<wire x1="3.9" y1="30.9" x2="5.1" y2="29.7" width="0.4064" layer="1"/>
-<via x="5.1" y="29.7" extent="1-16" drill="0.6" diameter="1.4224" shape="square"/>
-<wire x1="9.6" y1="25.2" x2="5.1" y2="29.7" width="0.4064" layer="16"/>
 <wire x1="6.6" y1="19" x2="6.6" y2="9" width="0.4064" layer="16"/>
 <wire x1="6.6" y1="9" x2="8.5" y2="7.1" width="0.4064" layer="16"/>
@@
 <wire x1="37.5" y1="17.1" x2="37.5" y2="19" width="0.4064" layer="16"/>
 <wire x1="37.5" y1="19" x2="38.7" y2="20.2" width="0.4064" layer="16"/>
-<wire x1="5.1" y1="29.7" x2="5.1" y2="29.8" width="0.4064" layer="16"/>
-<wire x1="5.1" y1="29.8" x2="8.2" y2="32.9" width="0.4064" layer="16"/>
-<via x="8.2" y="34.5" extent="1-16" drill="0.6" diameter="1.4224" shape="square"/>
-<wire x1="8.2" y1="32.9" x2="8.2" y2="34.5" width="0.4064" layer="16"/>
-<wire x1="8.2" y1="34.5" x2="10.1" y2="34.5" width="0.4064" layer="1"/>
-<wire x1="8.2" y1="32.9" x2="11" y2="30.1" width="0.4064" layer="16"/>
-<wire x1="11" y1="30.1" x2="12.2" y2="30.1" width="0.4064" layer="16"/>
-<wire x1="9.6" y1="24" x2="15.1" y2="18.5" width="0.4064" layer="16"/>
-<wire x1="15.1" y1="18.5" x2="15.2" y2="12.4" width="0.4064" layer="16"/>
-<via x="15.2" y="12.4" extent="1-16" drill="0.6" diameter="1.4224" shape="square"/>
-<wire x1="12.4" y1="12.5" x2="15.1" y2="12.5" width="0.4064" layer="1"/>
-<wire x1="15.1" y1="12.5" x2="15.2" y2="12.4" width="0.4064" layer="1"/>
 <wire x1="40" y1="26.8" x2="38.1" y2="26.8" width="0.4064" layer="1"/>
-<polygon width="0.4064" layer="1">
-<vertex x="2" y="79"/>
-<vertex x="53" y="79"/>
-<vertex x="53" y="2"/>
-<vertex x="2" y="2"/>
-</polygon>
-<polygon width="0.4064" layer="16">
-<vertex x="2" y="79"/>
-<vertex x="53" y="79"/>
-<vertex x="53" y="2"/>
-<vertex x="2" y="2"/>
-</polygon>
-<wire x1="15.2" y1="12.4" x2="19.5" y2="12.4" width="0.4064" layer="1"/>
-<wire x1="19.5" y1="12.4" x2="19.9" y2="12" width="0.4064" layer="1"/>
 <wire x1="16.8" y1="80.1" x2="16" y2="79.3" width="0.4064" layer="1"/>
 <wire x1="16" y1="79.3" x2="16" y2="76.9" width="0.4064" layer="1"/>
@@
 <wire x1="1.9" y1="72.4" x2="4.4" y2="72.4" width="0.4064" layer="1"/>
 <wire x1="4.4" y1="72.4" x2="4.5" y2="72.5" width="0.4064" layer="1"/>
+<wire x1="42.4" y1="33" x2="42.4" y2="32.5" width="0" layer="19" extent="1-1"/>
+<wire x1="6.6" y1="19" x2="10.6" y2="19" width="0.4064" layer="16"/>
+<wire x1="10.6" y1="19" x2="11.9" y2="20.3" width="0.4064" layer="16"/>
+<wire x1="19.5" y1="12.4" x2="19.9" y2="12" width="0.4064" layer="1"/>
+<wire x1="13.3" y1="20.3" x2="14.2" y2="19.4" width="0.4064" layer="16"/>
+<wire x1="14.2" y1="19.4" x2="15.1" y2="18.5" width="0.4064" layer="16"/>
+<wire x1="15.1" y1="18.5" x2="15.2" y2="12.4" width="0.4064" layer="16"/>
+<via x="15.2" y="12.4" extent="1-16" drill="0.6" diameter="1.4224" shape="square"/>
+<wire x1="15.2" y1="12.4" x2="19.5" y2="12.4" width="0.4064" layer="1"/>
+<wire x1="15.1" y1="12.5" x2="15.2" y2="12.4" width="0.4064" layer="1"/>
+<wire x1="12.4" y1="12.5" x2="15.1" y2="12.5" width="0.4064" layer="1"/>
+<wire x1="11.9" y1="20.3" x2="13.3" y2="20.3" width="0.4064" layer="16"/>
+<wire x1="11" y1="30.1" x2="12.2" y2="30.1" width="0.4064" layer="16"/>
+<wire x1="8.2" y1="34.5" x2="10.1" y2="34.5" width="0.4064" layer="1"/>
+<via x="8.2" y="34.5" extent="1-16" drill="0.6" diameter="1.4224" shape="square"/>
+<wire x1="8.2" y1="32.9" x2="8.2" y2="34.5" width="0.4064" layer="16"/>
+<wire x1="8.2" y1="32.9" x2="11" y2="30.1" width="0.4064" layer="16"/>
+<wire x1="5.1" y1="29.8" x2="8.2" y2="32.9" width="0.4064" layer="16"/>
+<wire x1="3.9" y1="32.1" x2="3.9" y2="30.9" width="0.4064" layer="1"/>
+<wire x1="3.9" y1="30.9" x2="5.1" y2="29.7" width="0.4064" layer="1"/>
+<via x="5.1" y="29.7" extent="1-16" drill="0.6" diameter="1.4224" shape="square"/>
+<wire x1="5.1" y1="29.7" x2="5.1" y2="29.8" width="0.4064" layer="16"/>
+<wire x1="5.1" y1="29.7" x2="8.8" y2="29.7" width="0.4064" layer="16"/>
+<wire x1="8.8" y1="29.7" x2="12.1" y2="26.4" width="0.4064" layer="16"/>
+<wire x1="12.1" y1="26.4" x2="12.1" y2="21.5" width="0.4064" layer="16"/>
+<wire x1="12.1" y1="21.5" x2="13.3" y2="20.3" width="0.4064" layer="16"/>
 </signal>
 <signal name="S$6">
@@
 <wire x1="52.9" y1="68.7" x2="52.1" y2="69.5" width="0.4064" layer="1"/>
 <wire x1="52.1" y1="69.5" x2="47.9" y2="69.5" width="0.4064" layer="1"/>
-</signal>
-<signal name="S$16">
-<wire x1="3.4" y1="24" x2="3.4" y2="20.9" width="0.4064" layer="16"/>
-<wire x1="3.4" y1="20.9" x2="3.1" y2="20.6" width="0.4064" layer="16"/>
-<wire x1="3.1" y1="20.6" x2="3.1" y2="16.6" width="0.4064" layer="16"/>
-<wire x1="3.1" y1="16.6" x2="3.1" y2="15.7" width="0.4064" layer="16"/>
-<wire x1="3.1" y1="15.7" x2="3.1" y2="15.2" width="0.4064" layer="16"/>
-<wire x1="3.1" y1="15.2" x2="3" y2="15.1" width="0.4064" layer="16"/>
 </signal>
 <signal name="S$2">
@@
 </signal>
 <signal name="S$13">
-<wire x1="24.4" y1="76.3" x2="24.4" y2="76" width="0.4064" layer="16"/>
-<wire x1="24.4" y1="76" x2="25.7" y2="74.7" width="0.4064" layer="16"/>
-<wire x1="25.7" y1="74.7" x2="25.7" y2="71.7" width="0.4064" layer="16"/>
-<wire x1="25.7" y1="71.7" x2="25.3" y2="71.3" width="0.4064" layer="16"/>
+<wire x1="24.4" y1="76.3" x2="24.4" y2="75.9" width="0.4064" layer="16"/>
+<wire x1="25.8" y1="71.8" x2="25.3" y2="71.3" width="0.4064" layer="16"/>
 <wire x1="25.3" y1="71.3" x2="23.8" y2="71.3" width="0.4064" layer="16"/>
 <wire x1="23.8" y1="71.3" x2="22" y2="69.5" width="0.4064" layer="16"/>
@@
 <wire x1="30.7" y1="68.3" x2="30.8" y2="68.2" width="0.4064" layer="16"/>
 <wire x1="30.8" y1="68.2" x2="30.8" y2="66.8" width="0.4064" layer="16"/>
+<wire x1="25.8" y1="71.8" x2="25.8" y2="74.5" width="0.3048" layer="16"/>
+<wire x1="25.8" y1="74.5" x2="24.4" y2="75.9" width="0.3048" layer="16"/>
 </signal>
 <signal name="S$22">
@@
 <wire x1="32.1" y1="46.6" x2="32.1" y2="44.2" width="0.4064" layer="1"/>
 </signal>
+<signal name="S$89">
+<wire x1="9.6" y1="24" x2="9.6" y2="25.6" width="0.4064" layer="16"/>
+<wire x1="9.6" y1="25.6" x2="7.5" y2="27.7" width="0.4064" layer="16"/>
+<wire x1="7.5" y1="27.7" x2="2.3" y2="27.7" width="0.4064" layer="16"/>
+<wire x1="2.3" y1="27.7" x2="1.2" y2="26.6" width="0.4064" layer="16"/>
+<wire x1="1.2" y1="26.6" x2="1.2" y2="16.9" width="0.4064" layer="16"/>
+<wire x1="1.2" y1="16.9" x2="3" y2="15.1" width="0.4064" layer="16"/>
+</signal>
 </signals>
